File: hardware_rf/hardware_rf.kicad_sch (KiCad schematic)
At the start: 5 parts, among them IC1 CC1125RHBR, Y1 Crystal_GND24

Commit message: schematic work
Parts:
- added C10: 10n, symbol Device:C
- added C11, C12, C13, C15, C16, C3, C4, C5, C6, C7, C9: 47n, symbol Device:C
- added C14: 220n, symbol Device:C
- added C8: 1n8, symbol Device:C
- added R2: 56k, symbol Device:R
- C1, C2: value C -> 15p
Connections:
- net GND: now also C10.2, C11.2, C12.2, C13.2, C14.2, C15.2, C16.1, C3.1, C4.1, C5.1, C6.1, C7.1, C9.2, R2.2
- net at IC1.1 (VDD_GUARD): now also C16.2
- net GPIO0: now reaches IC1.10 (GPIO0)
- net CSN: now reaches IC1.11 (CSN)
- net 3v3: now reaches IC1.12 (DVDD_2)
- net 3v3: now also IC1.13 (AVDD_IF), IC1.15 (AVDD_RF), IC1.22 (AVDD_SYNTH1), IC1.25 (AVDD_PFD_CHP), IC1.27 (AVDD_SYNTH2), IC1.28 (AVDD_XOSC), C11.1, C12.1, C13.1, C4.2, C5.2, C7.2, C9.1
- net at IC1.14 (RBIAS): now also R2.1
- net PA: now reaches IC1.17 (PA)
- net TRX_SW: now reaches IC1.18 (TRX_SW)
- net LNA_P: now reaches IC1.19 (LNA_P)
- net RSTN: now reaches IC1.2 (RESET_N)
- net LNA_N: now reaches IC1.20 (LNA_N)
- net at IC1.21 (DCPL_VCO): now also C10.1
- net at IC1.23 (LPF0): now also C8.2
- net at IC1.24 (LPF1): now also C8.1
- net at IC1.26 (DCPL_PFD_CHP): now also C6.2
- net at IC1.29 (DCPL_XOSC): now also C3.2
- net GPIO3: now reaches IC1.3 (GPIO3)
- net GPIO2: now reaches IC1.4 (GPIO2)
- net at IC1.5 (DVDD_1): now also C15.1
- net at IC1.6 (DCPL): now also C14.1
- net MOSI: now reaches IC1.7 (SI)
- net SCLK: now reaches IC1.8 (SCLK)
- net MISO: now reaches IC1.9 (SO(GPIO1))
Other:
- note added: "U2J"
- note added: "X5R"
- note added: "X7R"
- moved on the sheet: C1, C2, IC1, R1, Y1

Commit message: pcb
Parts:
- added C17, C18, C19, C21: 4.7u, symbol Device:C
- added C20, C22, C23, C24, C25, C26, C27, C28, C29, C30, C31: 100n, symbol Device:C
- added C32, C33: 15p, symbol Device:C
- added L1: 3.3u, symbol Device:L
- added R3: 33, symbol Device:R
- added R4, R5: 27, symbol Device:R
- added R6: R, symbol Device:R
- added R7: 1k, symbol Device:R
- added SW1: SW_Push, symbol Switch:SW_Push
- added U1: RP2350A-QFN60, mainfoot:RP2350A_QFN-60_EP_7.75x7.75_Pitch0.4mm, symbol mainlib:RP2350A-QFN60
- added U2: W25Q128JVS, Package_SO:SOIC-8_5.3x5.3mm_P1.27mm, symbol Memory_Flash:W25Q128JVS
- added Y2: Crystal_GND24, symbol Device:Crystal_GND24
Connections:
- net 3v3: now also C17.1, C23.1, C24.1, C25.1, C26.1, C27.1, C28.1, C29.1, C30.1, C31.1, R3.1, U1.1 (IOVDD), U1.11 (IOVDD), U1.20 (IOVDD), U1.30 (IOVDD), U1.38 (IOVDD), U1.44 (ADC_AVDD), U1.45 (IOVDD), U1.49 (VREG_VIN), U1.53 (USB_OTP_VDD), U1.54 (QSPI_IOVDD), U2.8 (VCC)
- net GND: now also C17.2, C18.2, C19.2, C20.2, C21.2, C22.2, C23.2, C24.2, C25.2, C26.2, C27.2, C28.2, C29.2, C30.2, C31.2, C32.1, C33.1, SW1.2, U1.47 (VREG_PGND), U1.61 (GND), U2.4 (GND), Y2.2, Y2.4
- new net: R7.2, U1.22 (XOUT)
- new net: C18.1, R3.2, U1.46 (VREG_AVDD)
- new net: L1.2, U1.48 (VREG_LX)
- new net: R4.1, U1.51 (USB_DM)
- new net: R5.1, U1.52 (USB_DP)
- new net: R6.1, SW1.1
- new net 1v1: C19.1, C20.1, C21.1, C22.1, L1.1, U1.23 (DVDD), U1.39 (DVDD), U1.50 (VREG_FB), U1.6 (DVDD)
- new net QSPI_SCLK: U1.56 (QSPI_SCLK), U2.6 (CLK)
- new net QSPI_SD0: U1.57 (QSPI_SD0), U2.5 (DI/IO_{0})
- new net QSPI_SD1: U1.59 (QSPI_SD1), U2.2 (DO/IO_{1})
- new net QSPI_SD2: U1.58 (QSPI_SD2), U2.3 (~{WP}/IO_{2})
- new net QSPI_SD3: U1.55 (QSPI_SD3), U2.7 (~{HOLD}/~{RESET}/IO_{3})
- new net QSPI_SS: R6.2, U1.60 (QSPI_SS), U2.1 (~{CS})
- new net USB_DM: R4.2
- new net USB_DP: R5.2
- new net XIN: C33.2, U1.21 (XIN), Y2.1
- new net XOUT: C32.2, R7.1, Y2.3
Other:
- title: (none) -> RF Board For VikramSAT
- moved on the sheet: C1, C10, C11, C12, C13, C14, C15, C16, C2, C3, C4, C5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

Commit message: journaling
Parts:
- added J1: Conn_Coaxial, symbol Connector:Conn_Coaxial
Changed lines of the file:
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@@
+	)
+	(symbol
+		(lib_id "Connector:Conn_Coaxial")
+		(at 207.01 234.95 0)
+		(unit 1)
+		(exclude_from_sim no)
+		(in_bom yes)
+		(on_board yes)
+		(dnp no)
+		(fields_autoplaced yes)
+		(property "Reference" "J1"
+			(at 210.82 233.9731 0)
+			(effects
+				(font
+					(size 1.27 1.27)
+				)
+				(justify left)
+			)
+		)
+		(property "Value" "Conn_Coaxial"
+			(at 210.82 236.5131 0)
+			(effects
+				(font
+					(size 1.27 1.27)
+				)
+				(justify left)
+			)
+		)
+		(property "Footprint" ""
+			(at 207.01 234.95 0)
+			(effects
+				(font
+					(size 1.27 1.27)
+				)
+				(hide yes)
+			)
+		)
+		(property "Datasheet" "~"
+			(at 207.01 234.95 0)
+			(effects
+				(font
+					(size 1.27 1.27)
+				)
+				(hide yes)
+			)
+		)
+		(property "Description" "coaxial connector (BNC, SMA, SMB, SMC, Cinch/RCA, LEMO, ...)"
+			(at 207.01 234.95 0)
+			(effects
+				(font
+					(size 1.27 1.27)
+				)
+				(hide yes)
+			)
+		)
+		(pin "2"
+		)
+		(pin "1"
+		)
+		(instances
+			(project ""
+				(path "/76e9da14-bca7-4795-80b8-b5efcf73ac31"
+					(reference "J1")
+					(unit 1)
+				)
+			)
+		)
 	)
 	(symbol

Commit message: symbol
Parts:
- added DP1: ~, mainfoot:Debug Pad, symbol mainlib:Debug_Pads
- added J2: Conn_01x03_Socket, symbol Connector:Conn_01x03_Socket
Connections:
- net GND: now also J2.2 (Pin_2)
- net at U1.24 (SWCLK): now also J2.3 (Pin_3)
- net at U1.25 (SWDIO): now also J2.1 (Pin_1)
Changed lines of the file:
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@@
 	(wire
 		(pts
+			(xy 182.88 135.89) (xy 196.85 135.89)
+		)
+		(stroke
+			(width 0)
+			(type default)
+		)
+	)
+	(wire
+		(pts
 			(xy 180.34 76.2) (xy 196.85 76.2)
 		)
@@
 	(wire
 		(pts
+			(xy 196.85 137.16) (xy 196.85 135.89)
+		)
+		(stroke
+			(width 0)
+			(type default)
+		)
+	)
+	(wire
+		(pts
 			(xy 63.5 74.93) (xy 68.58 74.93)
 		)
@@
 	(wire
 		(pts
+			(xy 182.88 140.97) (xy 196.85 140.97)
+		)
+		(stroke
+			(width 0)
+			(type default)
+		)
+	)
+	(wire
+		(pts
 			(xy 240.03 62.23) (xy 243.84 62.23)
 		)
@@
 	(wire
 		(pts
+			(xy 196.85 140.97) (xy 196.85 139.7)
+		)
+		(stroke
+			(width 0)
+			(type default)
+		)
+	)
+	(wire
+		(pts
 			(xy 279.4 48.26) (xy 288.29 48.26)
 		)
@@
 	(global_label "GND"
 		(shape input)
+		(at 182.88 138.43 0)
+		(fields_autoplaced yes)
+		(effects
+			(font
+				(size 1.27 1.27)
+			)
+			(justify left)
+		)
+		(property "Intersheetrefs" "${INTERSHEET_REFS}"
+			(at 189.7357 138.43 0)
+			(effects
+				(font
+					(size 1.27 1.27)
+				)
+				(justify left)
+				(hide yes)
+			)
+		)
+	)
+	(global_label "GND"
+		(shape input)
 		(at 120.65 207.01 270)
 		(fields_autoplaced yes)
@@
 	)
 	(symbol
+		(lib_id "Connector:Conn_01x03_Socket")
+		(at 177.8 138.43 180)
+		(unit 1)
+		(exclude_from_sim no)
+		(in_bom yes)
+		(on_board yes)
+		(dnp no)
+		(fields_autoplaced yes)
+		(property "Reference" "J2"
+			(at 178.435 130.81 0)
+			(effects
+				(font
+					(size 1.27 1.27)
+				)
+			)
+		)
+		(property "Value" "Conn_01x03_Socket"
+			(at 178.435 133.35 0)
+			(effects
+				(font
+					(size 1.27 1.27)
+				)
+			)
+		)
+		(property "Footprint" ""
+			(at 177.8 138.43 0)
+			(effects
+				(font
+					(size 1.27 1.27)
+				)
+				(hide yes)
+			)
+		)
+		(property "Datasheet" "~"
+			(at 177.8 138.43 0)
+			(effects
+				(font
+					(size 1.27 1.27)
+				)
+				(hide yes)
+			)
+		)
+		(property "Description" "Generic connector, single row, 01x03, script generated"
+			(at 177.8 138.43 0)
+			(effects
+				(font
+					(size 1.27 1.27)
+				)
+				(hide yes)
+			)
+		)
+		(pin "3"
+		)
+		(pin "2"
+		)
+		(pin "1"
+		)
+		(instances
+			(project ""
+				(path "/76e9da14-bca7-4795-80b8-b5efcf73ac31"
+					(reference "J2")
+					(unit 1)
+				)
+			)
+		)
+	)
+	(symbol
 		(lib_id "Device:C")
 		(at 200.66 44.45 0)
@@
 					(unit 1)
 				)
+			)
+		)
+	)
+	(symbol
+		(lib_id "mainlib:Debug_Pads")
+		(at 158.75 171.45 0)
+		(unit 1)
+		(exclude_from_sim no)
+		(in_bom yes)
+		(on_board yes)
+		(dnp no)
+		(fields_autoplaced yes)
+		(property "Reference" "DP1"
+			(at 158.75 165.1 0)
+			(effects
+				(font
+					(size 1.27 1.27)
+				)
+			)
+		)
+		(property "Value" "~"
+			(at 158.75 167.64 0)
+			(effects
+				(font
+					(size 1.27 1.27)
+				)
+			)
+		)
+		(property "Footprint" "mainfoot:Debug Pad"
+			(at 158.75 171.45 0)
+			(effects
+				(font
+					(size 1.27 1.27)
+				)
+				(hide yes)
+			)
+		)
+		(property "Datasheet" ""
+			(at 158.75 171.45 0)
+			(effects
+				(font
+					(size 1.27 1.27)
+				)
+				(hide yes)
+			)
+		)
+		(property "Description" ""
+			(at 158.75 171.45 0)
+			(effects
+				(font
+					(size 1.27 1.27)
+				)
+				(hide yes)
+			)
+		)
+		(pin "2"
+		)
+		(pin "1"
+		)
+		(instances
+			(project ""
+				(path "/76e9da14-bca7-4795-80b8-b5efcf73ac31"
+					(reference "DP1")
+					(unit 1)
+				)

Commit message: pcb
Parts:
- added DP2, DP3, DP4, DP5: ~, mainfoot:Debug Pad, symbol mainlib:Debug_Pads
- added IC2: BALF-SPI2-02D3, mainfoot:BALFSPI202D3, symbol mainlib:BALF-SPI2-02D3
- added IC3: 4259-63, mainfoot:PE4259, symbol mainlib:4259-63
- added R10, R8, R9: R, symbol Device:R
- added R11: 10k, symbol Device:R
Connections:
- net 3v3: now also DP5.1 (Pin1), IC3.6 (~{CTRL_OR_VDD}), R10.2
- net CSN: now also DP4.2 (Pin2)
- net GND: now also J1.2 (Ext), DP5.2 (Pin2), IC2.4 (GND_1), IC2.6 (GND_2), R8.1, R9.2
- net GPIO0: now also DP2.2 (Pin2)
- net GPIO2: now also DP2.1 (Pin1)
- net GPIO3: now also DP1.2 (Pin2)
- net LNA_N: now also IC2.2 (RXN), R9.1
- net LNA_P: now also IC2.1 (RXP), R8.2
- net MISO: now also DP3.1 (Pin1)
- net MOSI: now also DP3.2 (Pin2)
- net PA: now also IC2.3 (TX), R10.1
- net RSTN: now also DP1.1 (Pin1)
- net SCLK: now also DP4.1 (Pin1)
- net TRX_SW: now also R11.1
- net ANT: now reaches J1.1 (In)
- new net: IC2.5 (ANT), IC3.5 (RFC)
- new net CTRL: IC3.4 (CTRL)
Other:
- note added: "Route as 50R"
- moved on the sheet: DP1, J1

Commit message: pcb
Connections:
- net CTRL: now also IC2.5 (ANT), IC3.5 (RFC)
Changed lines of the file:
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@@
+		)
+	)
+	(global_label "CTRL"
+		(shape input)
+		(at 255.27 210.82 180)
+		(fields_autoplaced yes)
+		(effects
+			(font
+				(size 1.27 1.27)
+			)
+			(justify right)
+		)
+		(property "Intersheetrefs" "${INTERSHEET_REFS}"
+			(at 247.7491 210.82 0)
+			(effects
+				(font
+					(size 1.27 1.27)
+				)
+				(justify right)
+				(hide yes)
+			)
 		)
 	)

Commit message: symbol
Connections:
- net CTRL: no longer IC2.5 (ANT), IC3.5 (RFC)
- net GND: now also IC3.2 (GND)
- new net: IC2.5 (ANT), IC3.5 (RFC)
Other:
- moved on the sheet: IC2, IC3, R10, R6, R8, R9, SW1, U2

Commit message: sch
Parts:
- added IC4: 4259-63, mainfoot:PE4259, symbol mainlib:4259-63
- added U3: GSQ5111, easyeda2kicad:QFN-16_L3.0-W3.0-P0.50-TL-EP1.65, symbol easyeda2kicad:GSQ5111
- added U4: SK5129, easyeda2kicad:DFN-6_L1.6-W1.6-P0.50-BL-EP1.0, symbol easyeda2kicad:SK5129
Connections:
- net 3v3: now also IC4.6 (~{CTRL_OR_VDD}), U4.1 (VDD), U4.6 (VDD)
- net CTRL: now also IC4.4 (CTRL)
- net GND: now also IC4.2 (GND), U3.1 (GND), U3.14 (GND), U3.3 (GND), U3.8 (GND), U4.2 (GND), U4.7 (EP)
- net at IC3.1 (RF1): now also U4.3 (LNA_IN)
- net at IC3.3 (RF2): now also U3.2 (RF_IN)
- net ANT: no longer names the net of J1.1 (In)
- net ANT: now also IC4.5 (RFC)
- new net: IC4.3 (RF2), U3.10 (RF_OUT), U3.11 (RF_OUT), U3.12 (RF_OUT), U3.9 (RF_OUT)
- new net: IC4.1 (RF1), U4.5 (LNA_OUT)
- new net LNA_PD_EN: U4.4 (PD_EN)
Other:
- moved on the sheet: J1
