File: hardware_rf/hardware_rf.kicad_pcb (KiCad board)
At the start: 4 copper layers, 72 x 72 mm, 90 parts, among them IC1 CC1125RHBR, IC2 BALF-SPI2-02D3, IC3 4259-63, IC4 4259-63, J1 Conn_Coaxial, J2 Conn_01x03_Socket, J3 Conn_02x20_Top_Bottom, J4 USB_C_Receptacle_USB2.0_16P, SW1 SW_Push, U1 RP2350A-QFN60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

Commit message: pcb
Parts:
- moved R12 24.2 mm to (135.9, 115.8), turned to 180 degrees
- moved C30 21.4 mm to (156.6, 119.2), turned to 0 degrees
- moved C27 16.5 mm to (156.6, 115.0), turned to 0 degrees
- moved C22 15.7 mm to (140.3, 118.0), turned to 180 degrees
- moved C29 10.3 mm to (150.9, 108.1), turned to 90 degrees
- moved C21 9.55 mm to (147.7, 108.1), turned to 90 degrees
- moved C25 7.00 mm to (140.3, 121.9)
- moved C28 5.73 mm to (146.3, 108.1), turned to 90 degrees
- moved D1 4.23 mm to (138.4, 115.8), turned to 0 degrees
- moved C26 3.63 mm to (142.6, 109.8), turned to 90 degrees
- moved U2 3.32 mm to (155.6, 127.0)
- moved SW1 1.85 mm to (162.7, 122.0)
- moved C20 1.58 mm to (156.6, 117.0)
- moved C23 0.90 mm to (140.3, 119.7)
- moved R7 0.75 mm to (149.0, 108.1)
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Routing:
- net 3v3: track 0.00 -> 35.2 mm
- net 1v1: track 0.00 -> 33.1 mm
- net QSPI_SS: track 0.00 -> 17.4 mm
- net QSPI_SD1: track 0.00 -> 16.0 mm
- net QSPI_SD2: track 0.00 -> 12.2 mm
- net QSPI_SD3: track 0.00 -> 9.62 mm
- net XIN: track 0.00 -> 9.28 mm
- net Net-(R6-Pad1): track 0.00 -> 8.92 mm
- net QSPI_SCLK: track 0.00 -> 8.33 mm
- net QSPI_SD0: track 0.00 -> 6.33 mm
- net Net-(D1-A): track 0.00 -> 6.11 mm
- net Net-(U1-VREG_LX): track 0.00 -> 4.93 mm
- net Net-(U1-VREG_AVDD): track 0.00 -> 4.52 mm
- net Net-(U1-XOUT): track 0.00 -> 4.20 mm
- net GND: track 0.00 -> 3.34 mm
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
Commit message: pcb
Parts:
- moved C42 10.1 mm to (172.8, 129.8)
- moved C41 9.04 mm to (172.7, 133.4)
- moved C11 3.91 mm to (165.3, 113.0)
- moved R2 3.91 mm to (167.1, 113.0)
- moved C12 3.91 mm to (163.9, 112.9)
- moved C13 3.91 mm to (162.0, 112.9)
- moved D2 2.67 mm to (162.5, 133.4), turned to 180 degrees
- moved IC1 2.08 mm to (163.8, 105.0)
- moved J2 2.01 mm to (140.1, 84.7)
- moved D3 0.83 mm to (162.5, 131.9)
- moved R1 0.33 mm to (160.8, 100.8)
- moved C20 0.12 mm to (156.6, 117.2)
- moved C30 0.08 mm to (156.6, 119.3)
Routing:
- net 3v3: track 35.2 -> 39.5 mm
Changed lines of the file:
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@@
 	(footprint "Diode_SMD:D_0402_1005Metric"
 		(layer "F.Cu")
-		(at 162.4525 130.71)
+		(at 162.475 133.375 180)
 		(descr "Diode SMD 0402 (1005 Metric), square (rectangular) end terminal, IPC-7351 nominal, (Body size source: http://www.tortai-tech.com/upload/download/2011102023233369053.pdf), generated with kicad-footprint-generator")
 		(tags "diode")
@@
 		)
 		(property "Sim.Device" "D"
-			(at 0 0 0)
+			(at 0 0 180)
 			(unlocked yes)
 			(layer "F.Fab")
@@
 		)
 		(property "Sim.Pins" "1=K 2=A"
-			(at 0 0 0)
+			(at 0 0 180)
 			(unlocked yes)
 			(layer "F.Fab")
@@
 		)
 		(fp_line
-			(start -0.93 -0.47)
-			(end 0.93 -0.47)
+			(start 0.93 0.47)
+			(end -0.93 0.47)
 			(stroke
 				(width 0.05)
@@
 		)
 		(fp_line
-			(start -0.93 0.47)
-			(end -0.93 -0.47)
+			(start 0.93 -0.47)
+			(end 0.93 0.47)
 			(stroke
 				(width 0.05)
@@
 		)
 		(fp_line
-			(start 0.93 -0.47)
-			(end 0.93 0.47)
+			(start -0.93 0.47)
+			(end -0.93 -0.47)
 			(stroke
 				(width 0.05)
@@
 		)
 		(fp_line
-			(start 0.93 0.47)
-			(end -0.93 0.47)
+			(start -0.93 -0.47)
+			(end 0.93 -0.47)
 			(stroke
 				(width 0.05)
@@
 		)
 		(fp_line
-			(start -0.5 -0.25)
-			(end 0.5 -0.25)
+			(start 0.5 0.25)
+			(end -0.5 0.25)
 			(stroke
 				(width 0.1)
@@
 		)
 		(fp_line
-			(start -0.5 0.25)
-			(end -0.5 -0.25)
+			(start 0.5 -0.25)
+			(end 0.5 0.25)
 			(stroke
 				(width 0.1)
@@
 		)
 		(fp_line
-			(start -0.4 0.25)
-			(end -0.4 -0.25)
+			(start -0.3 0.25)
+			(end -0.3 -0.25)
 			(stroke
 				(width 0.1)
@@
 		)
 		(fp_line
-			(start -0.3 0.25)
-			(end -0.3 -0.25)
+			(start -0.4 0.25)
+			(end -0.4 -0.25)
 			(stroke
 				(width 0.1)
@@
 		)
 		(fp_line
-			(start 0.5 -0.25)
-			(end 0.5 0.25)
+			(start -0.5 0.25)
+			(end -0.5 -0.25)
 			(stroke
 				(width 0.1)
@@
 		)
 		(fp_line
-			(start 0.5 0.25)
-			(end -0.5 0.25)
+			(start -0.5 -0.25)
+			(end 0.5 -0.25)
 			(stroke
 				(width 0.1)
@@
 		)
 		(pad "1" smd roundrect
-			(at -0.485 0)
+			(at -0.485 0 180)
 			(size 0.59 0.64)
 			(layers "F.Cu" "F.Mask" "F.Paste")
@@
 		)
 		(pad "2" smd roundrect
-			(at 0.485 0)
+			(at 0.485 0 180)
 			(size 0.59 0.64)
 			(layers "F.Cu" "F.Mask" "F.Paste")
@@
 	(footprint "Capacitor_SMD:C_0805_2012Metric"
 		(layer "F.Cu")
-		(at 167.6125 125.975)
+		(at 172.725 133.425)
 		(descr "Capacitor SMD 0805 (2012 Metric), square (rectangular) end terminal, IPC-7351 nominal, (Body size source: IPC-SM-782 page 76, https://www.pcb-3d.com/wordpress/wp-content/uploads/ipc-sm-782a_amendment_1_and_2.pdf, https://docs.google.com/spreadsheets/d/1BsfQQcO9C6DZCsRaXUlFlo91Tg2WpOkGARC1WS5S8t0/edit?usp=sharing), generated with kicad-footprint-generator")
 		(tags "capacitor")
@@
 			(at 0 -1.68 0)
 			(layer "F.SilkS")
+			(hide yes)
 			(effects
 				(font
@@
 	(footprint "Capacitor_SMD:C_0402_1005Metric"
 		(layer "F.Cu")
-		(at 156.575 119.25)
+		(at 156.6 119.325)
 		(descr "Capacitor SMD 0402 (1005 Metric), square (rectangular) end terminal, IPC-7351 nominal, (Body size source: IPC-SM-782 page 76, https://www.pcb-3d.com/wordpress/wp-content/uploads/ipc-sm-782a_amendment_1_and_2.pdf), generated with kicad-footprint-generator")
 		(tags "capacitor")
@@
 	(footprint "mainfoot:QFN50P500X500X100-33N-D"
 		(layer "F.Cu")
-		(at 165.125 103.425)
+		(at 163.8 105.025)
 		(descr "RHB0032N-1")
 		(tags "Integrated Circuit")
@@
 	(footprint "Capacitor_SMD:C_0402_1005Metric"
 		(layer "F.Cu")
-		(at 160.575 109.295 -90)
+		(at 161.965 112.945 -90)
 		(descr "Capacitor SMD 0402 (1005 Metric), square (rectangular) end terminal, IPC-7351 nominal, (Body size source: IPC-SM-782 page 76, https://www.pcb-3d.com/wordpress/wp-content/uploads/ipc-sm-782a_amendment_1_and_2.pdf), generated with kicad-footprint-generator")
 		(tags "capacitor")
@@
 	(footprint "Capacitor_SMD:C_0805_2012Metric"
 		(layer "F.Cu")
-		(at 167.125 138.25)
+		(at 172.75 129.85)
 		(descr "Capacitor SMD 0805 (2012 Metric), square (rectangular) end terminal, IPC-7351 nominal, (Body size source: IPC-SM-782 page 76, https://www.pcb-3d.com/wordpress/wp-content/uploads/ipc-sm-782a_amendment_1_and_2.pdf, https://docs.google.com/spreadsheets/d/1BsfQQcO9C6DZCsRaXUlFlo91Tg2WpOkGARC1WS5S8t0/edit?usp=sharing), generated with kicad-footprint-generator")
 		(tags "capacitor")
@@
 			(at 0 -1.68 0)
 			(layer "F.SilkS")
+			(hide yes)
 			(effects
 				(font
@@
 	(footprint "Diode_SMD:D_0402_1005Metric"
 		(layer "F.Cu")
-		(at 162.4525 132.7)
+		(at 162.5 131.875)
 		(descr "Diode SMD 0402 (1005 Metric), square (rectangular) end terminal, IPC-7351 nominal, (Body size source: http://www.tortai-tech.com/upload/download/2011102023233369053.pdf), generated with kicad-footprint-generator")
 		(tags "diode")
@@
 	(footprint "Resistor_SMD:R_0402_1005Metric"
 		(layer "F.Cu")
-		(at 160.81 101.15)
+		(at 160.75 100.825)
 		(descr "Resistor SMD 0402 (1005 Metric), square (rectangular) end terminal, IPC-7351 nominal, (Body size source: IPC-SM-782 page 72, https://www.pcb-3d.com/wordpress/wp-content/uploads/ipc-sm-782a_amendment_1_and_2.pdf), generated with kicad-footprint-generator")
 		(tags "resistor")
@@
 	(footprint "Capacitor_SMD:C_0402_1005Metric"
 		(layer "F.Cu")
-		(at 163.95 109.375 -90)
+		(at 165.34 113.025 -90)
 		(descr "Capacitor SMD 0402 (1005 Metric), square (rectangular) end terminal, IPC-7351 nominal, (Body size source: IPC-SM-782 page 76, https://www.pcb-3d.com/wordpress/wp-content/uploads/ipc-sm-782a_amendment_1_and_2.pdf), generated with kicad-footprint-generator")
 		(tags "capacitor")
@@
 	(footprint "Capacitor_SMD:C_0402_1005Metric"
 		(layer "F.Cu")
-		(at 156.625 117.025)
+		(at 156.625 117.15)
 		(descr "Capacitor SMD 0402 (1005 Metric), square (rectangular) end terminal, IPC-7351 nominal, (Body size source: IPC-SM-782 page 76, https://www.pcb-3d.com/wordpress/wp-content/uploads/ipc-sm-782a_amendment_1_and_2.pdf), generated with kicad-footprint-generator")
 		(tags "capacitor")
@@
 	(footprint "Resistor_SMD:R_0402_1005Metric"
 		(layer "F.Cu")
-		(at 165.75 109.35)
+		(at 167.14 113)
 		(descr "Resistor SMD 0402 (1005 Metric), square (rectangular) end terminal, IPC-7351 nominal, (Body size source: IPC-SM-782 page 72, https://www.pcb-3d.com/wordpress/wp-content/uploads/ipc-sm-782a_amendment_1_and_2.pdf), generated with kicad-footprint-generator")
 		(tags "resistor")
@@
 			(at 0 -3.5 0)
 			(layer "F.SilkS")
+			(hide yes)
 			(effects
 				(font
@@
 	(footprint "Connector_PinHeader_2.54mm:PinHeader_1x03_P2.54mm_Vertical"
 		(layer "F.Cu")
-		(at 140.285 86.7 90)
+		(at 140.085 84.7 90)
 		(descr "Through hole straight pin header, 1x03, 2.54mm pitch, single row")
 		(tags "Through hole pin header THT 1x03 2.54mm single row")
@@
 	(footprint "Capacitor_SMD:C_0402_1005Metric"
 		(layer "F.Cu")
-		(at 162.545 109.295 -90)
+		(at 163.935 112.945 -90)
 		(descr "Capacitor SMD 0402 (1005 Metric), square (rectangular) end terminal, IPC-7351 nominal, (Body size source: IPC-SM-782 page 76, https://www.pcb-3d.com/wordpress/wp-content/uploads/ipc-sm-782a_amendment_1_and_2.pdf), generated with kicad-footprint-generator")
 		(tags "capacitor")
@@
 		(width 0.2)
 		(layer "F.Cu")
+		(net 5)
+	)
+	(segment
+		(start 156.145 114.975)
+		(end 151.825 114.975)
+		(width 0.2)
+		(layer "F.Cu")

Commit message: pcb
Parts:
- moved C11 4.57 mm to (167.5, 109.0), turned to 0 degrees
- moved R2 2.75 mm to (167.5, 110.3)
- moved C16 1.71 mm to (156.0, 103.2)
- moved C15 1.65 mm to (156.0, 105.0)
- moved R10 1.63 mm to (169.0, 107.3), turned to -90 degrees
- moved C14 0.69 mm to (156.0, 106.0)
Routing:
- net 3v3: track 39.5 -> 45.0 mm
- net Net-(IC1-RBIAS): track 0.00 -> 4.06 mm
Other:
- outline, holes or cut-outs redrawn
Changed lines of the file:
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@@
 			(at 0 -1.16 90)
 			(layer "F.SilkS")
+			(hide yes)
 			(effects
 				(font
@@
 	(footprint "Capacitor_SMD:C_0402_1005Metric"
 		(layer "F.Cu")
-		(at 156.155 105.325 180)
+		(at 156 106 180)
 		(descr "Capacitor SMD 0402 (1005 Metric), square (rectangular) end terminal, IPC-7351 nominal, (Body size source: IPC-SM-782 page 76, https://www.pcb-3d.com/wordpress/wp-content/uploads/ipc-sm-782a_amendment_1_and_2.pdf), generated with kicad-footprint-generator")
 		(tags "capacitor")
@@
 			(at 0 -1.16 0)
 			(layer "F.SilkS")
+			(hide yes)
 			(effects
 				(font
@@
 	(footprint "Capacitor_SMD:C_0402_1005Metric"
 		(layer "F.Cu")
-		(at 156.155 103.355 180)
+		(at 156 105 180)
 		(descr "Capacitor SMD 0402 (1005 Metric), square (rectangular) end terminal, IPC-7351 nominal, (Body size source: IPC-SM-782 page 76, https://www.pcb-3d.com/wordpress/wp-content/uploads/ipc-sm-782a_amendment_1_and_2.pdf), generated with kicad-footprint-generator")
 		(tags "capacitor")
@@
 			(at 0 -1.16 0)
 			(layer "F.SilkS")
+			(hide yes)
 			(effects
 				(font
@@
 	(footprint "Capacitor_SMD:C_0402_1005Metric"
 		(layer "F.Cu")
-		(at 165.34 113.025 -90)
+		(at 167.5 109)
 		(descr "Capacitor SMD 0402 (1005 Metric), square (rectangular) end terminal, IPC-7351 nominal, (Body size source: IPC-SM-782 page 76, https://www.pcb-3d.com/wordpress/wp-content/uploads/ipc-sm-782a_amendment_1_and_2.pdf), generated with kicad-footprint-generator")
 		(tags "capacitor")
 		(property "Reference" "C11"
-			(at 0 -1.16 90)
+			(at 0 -1.16 0)
 			(layer "F.SilkS")
+			(hide yes)
 			(effects
 				(font
@@
 		)
 		(property "Value" "47n"
-			(at 0 1.16 90)
+			(at 0 1.16 0)
 			(layer "F.Fab")
 			(effects
@@
 		)
 		(property "Datasheet" ""
-			(at 0 0 90)
+			(at 0 0 0)
 			(layer "F.Fab")
 			(hide yes)
@@
 		)
 		(property "Description" "Unpolarized capacitor"
-			(at 0 0 90)
+			(at 0 0 0)
 			(layer "F.Fab")
 			(hide yes)
@@
 		(attr smd)
 		(fp_line
-			(start -0.107836 0.36)
-			(end 0.107836 0.36)
+			(start -0.107836 -0.36)
+			(end 0.107836 -0.36)
 			(stroke
 				(width 0.12)
@@
 		)
 		(fp_line
-			(start -0.107836 -0.36)
-			(end 0.107836 -0.36)
+			(start -0.107836 0.36)
+			(end 0.107836 0.36)
 			(stroke
 				(width 0.12)
@@
 		)
 		(fp_line
-			(start -0.91 0.46)
-			(end -0.91 -0.46)
+			(start -0.91 -0.46)
+			(end 0.91 -0.46)
 			(stroke
 				(width 0.05)
@@
 		)
 		(fp_line
-			(start 0.91 0.46)
-			(end -0.91 0.46)
+			(start -0.91 0.46)
+			(end -0.91 -0.46)
 			(stroke
 				(width 0.05)
@@
 		)
 		(fp_line
-			(start -0.91 -0.46)
-			(end 0.91 -0.46)
+			(start 0.91 -0.46)
+			(end 0.91 0.46)
 			(stroke
 				(width 0.05)
@@
 		)
 		(fp_line
-			(start 0.91 -0.46)
-			(end 0.91 0.46)
+			(start 0.91 0.46)
+			(end -0.91 0.46)
 			(stroke
 				(width 0.05)
@@
 		)
 		(fp_line
-			(start -0.5 0.25)
-			(end -0.5 -0.25)
+			(start -0.5 -0.25)
+			(end 0.5 -0.25)
 			(stroke
 				(width 0.1)
@@
 		)
 		(fp_line
-			(start 0.5 0.25)
-			(end -0.5 0.25)
+			(start -0.5 0.25)
+			(end -0.5 -0.25)
 			(stroke
 				(width 0.1)
@@
 		)
 		(fp_line
-			(start -0.5 -0.25)
-			(end 0.5 -0.25)
+			(start 0.5 -0.25)
+			(end 0.5 0.25)
 			(stroke
 				(width 0.1)
@@
 		)
 		(fp_line
-			(start 0.5 -0.25)
-			(end 0.5 0.25)
+			(start 0.5 0.25)
+			(end -0.5 0.25)
 			(stroke
 				(width 0.1)
@@
 		)
 		(fp_text user "${REFERENCE}"
-			(at 0 0 90)
+			(at 0 0 0)
 			(layer "F.Fab")
 			(effects
@@
 		)
 		(pad "1" smd roundrect
-			(at -0.48 0 270)
+			(at -0.48 0)
 			(size 0.56 0.62)
 			(layers "F.Cu" "F.Mask" "F.Paste")
@@
 		)
 		(pad "2" smd roundrect
-			(at 0.48 0 270)
+			(at 0.48 0)
 			(size 0.56 0.62)
 			(layers "F.Cu" "F.Mask" "F.Paste")
@@
 	(footprint "Resistor_SMD:R_0402_1005Metric"
 		(layer "F.Cu")
-		(at 167.14 113)
+		(at 167.525 110.275)
 		(descr "Resistor SMD 0402 (1005 Metric), square (rectangular) end terminal, IPC-7351 nominal, (Body size source: IPC-SM-782 page 72, https://www.pcb-3d.com/wordpress/wp-content/uploads/ipc-sm-782a_amendment_1_and_2.pdf), generated with kicad-footprint-generator")
 		(tags "resistor")
@@
 			(at 0 -1.17 0)
 			(layer "F.SilkS")
+			(hide yes)
 			(effects
 				(font
@@
 	(footprint "Capacitor_SMD:C_0402_1005Metric"
 		(layer "F.Cu")
-		(at 156.22 101.55)
+		(at 156 103.25)
 		(descr "Capacitor SMD 0402 (1005 Metric), square (rectangular) end terminal, IPC-7351 nominal, (Body size source: IPC-SM-782 page 76, https://www.pcb-3d.com/wordpress/wp-content/uploads/ipc-sm-782a_amendment_1_and_2.pdf), generated with kicad-footprint-generator")
 		(tags "capacitor")
@@
 			(at 0 -1.16 90)
 			(layer "F.SilkS")
+			(hide yes)
 			(effects
 				(font
@@
 	(footprint "Resistor_SMD:R_0402_1005Metric"
 		(layer "F.Cu")
-		(at 170.625 107.15)
+		(at 169 107.275 -90)
 		(descr "Resistor SMD 0402 (1005 Metric), square (rectangular) end terminal, IPC-7351 nominal, (Body size source: IPC-SM-782 page 72, https://www.pcb-3d.com/wordpress/wp-content/uploads/ipc-sm-782a_amendment_1_and_2.pdf), generated with kicad-footprint-generator")
 		(tags "resistor")
 		(property "Reference" "R10"
-			(at 0 -1.17 0)
+			(at 0 -1.17 90)
 			(layer "F.SilkS")
 			(effects
@@
 		)
 		(property "Value" "10k"
-			(at 0 1.17 0)
+			(at 0 1.17 90)
 			(layer "F.Fab")
 			(effects
@@
 		)
 		(property "Datasheet" ""
-			(at 0 0 0)
+			(at 0 0 90)
 			(layer "F.Fab")
 			(hide yes)
@@
 		)
 		(property "Description" "Resistor"
-			(at 0 0 0)
+			(at 0 0 90)
 			(layer "F.Fab")
 			(hide yes)
@@
 		(attr smd)
 		(fp_line
-			(start -0.153641 -0.38)
-			(end 0.153641 -0.38)
+			(start -0.153641 0.38)
+			(end 0.153641 0.38)
 			(stroke
 				(width 0.12)
@@
 		)
 		(fp_line
-			(start -0.153641 0.38)
-			(end 0.153641 0.38)
+			(start -0.153641 -0.38)
+			(end 0.153641 -0.38)
 			(stroke
 				(width 0.12)
@@
 		)
 		(fp_line
-			(start -0.93 -0.47)
-			(end 0.93 -0.47)
+			(start -0.93 0.47)
+			(end -0.93 -0.47)
 			(stroke
 				(width 0.05)
@@
 		)
 		(fp_line
-			(start -0.93 0.47)
-			(end -0.93 -0.47)
+			(start 0.93 0.47)
+			(end -0.93 0.47)
 			(stroke
 				(width 0.05)
@@
 		)
 		(fp_line
-			(start 0.93 -0.47)
-			(end 0.93 0.47)
+			(start -0.93 -0.47)
+			(end 0.93 -0.47)
 			(stroke
 				(width 0.05)
@@
 		)
 		(fp_line
-			(start 0.93 0.47)
-			(end -0.93 0.47)
+			(start 0.93 -0.47)
+			(end 0.93 0.47)
 			(stroke
 				(width 0.05)
@@
 		)
 		(fp_line
-			(start -0.525 -0.27)
-			(end 0.525 -0.27)
+			(start -0.525 0.27)
+			(end -0.525 -0.27)
 			(stroke
 				(width 0.1)
@@
 		)
 		(fp_line
-			(start -0.525 0.27)
-			(end -0.525 -0.27)
+			(start 0.525 0.27)
+			(end -0.525 0.27)
 			(stroke
 				(width 0.1)
@@
 		)
 		(fp_line
-			(start 0.525 -0.27)
-			(end 0.525 0.27)
+			(start -0.525 -0.27)
+			(end 0.525 -0.27)
 			(stroke
 				(width 0.1)
@@
 		)
 		(fp_line
-			(start 0.525 0.27)
-			(end -0.525 0.27)
+			(start 0.525 -0.27)
+			(end 0.525 0.27)
 			(stroke
 				(width 0.1)
@@
 		)
 		(fp_text user "${REFERENCE}"
-			(at 0 0 0)
+			(at 0 0 90)
 			(layer "F.Fab")
 			(effects
@@
 		)
 		(pad "1" smd roundrect
-			(at -0.51 0)
+			(at -0.51 0 270)
 			(size 0.54 0.64)
 			(layers "F.Cu" "F.Mask" "F.Paste")
@@
 		)
 		(pad "2" smd roundrect
-			(at 0.51 0)
+			(at 0.51 0 270)
 			(size 0.54 0.64)
 			(layers "F.Cu" "F.Mask" "F.Paste")
@@
 		(layer "Edge.Cuts")
 	)
-	(gr_circle
-		(center 127.5 142)
-		(end 130.180954 140.653331)
-		(stroke
-			(width 0.05)
-			(type default)
-		)
-		(fill no)
-		(layer "Edge.Cuts")
-	)
 	(gr_line
 		(start 194.5 80)
@@
 	)
 	(segment
+		(start 165.05 107.475)
+		(end 165.05 108.152)
+		(width 0.2)
+		(layer "F.Cu")
+		(net 5)
+	)
+	(segment
 		(start 145.5875 112.7375)
 		(end 144.9875 112.7375)
@@
 	)
 	(segment
+		(start 165.898 109)
+		(end 167.02 109)
+		(width 0.2)
+		(layer "F.Cu")
+		(net 5)
+	)
+	(segment
 		(start 146.325 110.328907)
 		(end 146.325 109.285)
@@
 	)
 	(segment
+		(start 168.235 107.785)
+		(end 169 107.785)
+		(width 0.2)
+		(layer "F.Cu")
+		(net 5)
+	)
+	(segment
 		(start 148.3875 119.6125)
 		(end 148.7875 119.6125)
@@
 	)
 	(segment
+		(start 167.02 109)
+		(end 168.235 107.785)
+		(width 0.2)
+		(layer "F.Cu")
+		(net 5)
+	)
+	(segment
 		(start 140.805 121.75)
 		(end 143.125 124.07)
@@
 	)
 	(segment
+		(start 165.05 108.152)
+		(end 165.898 109)
+		(width 0.2)
+		(layer "F.Cu")
+		(net 5)
+	)
+	(segment
 		(start 143.125 121.975)
 		(end 143.125 123.05)
@@
 	)
 	(segment
+		(start 164.55 107.475)
+		(end 164.55 108.2191)
+		(width 0.2)
+		(layer "F.Cu")
+		(net 40)
+	)
+	(segment
+		(start 166.6059 110.275)
+		(end 167.015 110.275)
+		(width 0.2)
+		(layer "F.Cu")
+		(net 40)
+	)
+	(segment
+		(start 164.55 108.2191)
+		(end 166.6059 110.275)
+		(width 0.2)
+		(layer "F.Cu")
+		(net 40)
+	)
+	(segment

Commit message: Pcb Done
Parts:
- removed J2: Conn_01x03_Socket, Connector_PinHeader_2.54mm:PinHeader_1x03_P2.54mm_Vertical
- added G***: LOGO, LOGO, F.Cu at (0.00, 0.00)
- added G***: LOGO, LOGO, F.Cu at (168.5, 141.2)
- moved DP1 51.1 mm to (134.0, 109.7), turned to 0 degrees
- moved DP2 46.6 mm to (141.9, 101.5), turned to 0 degrees
- moved DP5 46.4 mm to (135.1, 130.3), turned to 0 degrees
- moved DP3 44.8 mm to (135.2, 123.1), turned to 0 degrees
- moved DP4 43.4 mm to (138.2, 109.7), turned to 180 degrees
- moved C48 37.8 mm to (173.2, 126.2), turned to -90 degrees
- moved C47 36.6 mm to (169.1, 116.6), turned to -90 degrees
- moved C46 33.9 mm to (174.0, 117.2)
- moved IC4 33.8 mm to (179.6, 128.3)
- moved J1 32.8 mm to (189.0, 128.4), turned to 0 degrees
- moved C39 31.8 mm to (179.5, 116.1), turned to 90 degrees
- moved C40 30.3 mm to (180.6, 116.1), turned to 90 degrees
- moved C45 29.8 mm to (174.4, 108.2), turned to -90 degrees
- moved C49 29.4 mm to (181.7, 124.7), turned to -90 degrees
- moved U4 28.4 mm to (170.7, 123.1), turned to -90 degrees
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Connections:
- IC4 pad 5: unconnected-(IC4-RFC-Pad5) -> Net-(IC4-RFC)
- J1 pad 1: unconnected-(J1-In-Pad1) -> Net-(IC4-RFC)
- J3 pad 24: unconnected-(J3-Pin_24-Pad24) -> UART0_TX
- J3 pad 25: unconnected-(J3-Pin_25-Pad25) -> UART0_RX
- U1 pad 24: Net-(J2-Pin_3) -> unconnected-(U1-SWCLK-Pad24)
- U1 pad 25: Net-(J2-Pin_1) -> unconnected-(U1-SWDIO-Pad25)
- U1 pad 42: unconnected-(U1-GPIO28_ADC2-Pad42) -> UART0_TX
- U1 pad 43: unconnected-(U1-GPIO29_ADC3-Pad43) -> UART0_RX
Routing:
- net 5v: track 0.00 -> 134.3 mm, vias 0 -> 3
- net GPIO3: track 0.00 -> 67.5 mm, vias 0 -> 3
- net SPI1_DEV3: track 0.00 -> 66.7 mm
- net SPI1_DEV2: track 0.00 -> 65.6 mm
- net SPI0_MISO: track 0.00 -> 63.5 mm, vias 0 -> 3
- net SPI0_MOSI: track 0.00 -> 63.4 mm, vias 0 -> 3
- net SPI1_DEV1: track 0.00 -> 60.5 mm, vias 0 -> 1
- net 3v3: track 45.0 -> 104.3 mm, vias 0 -> 19
- net SPI1_MOSI: track 0.00 -> 52.4 mm, vias 0 -> 2
- net SPI1_MISO: track 0.00 -> 52.1 mm, vias 0 -> 1
- net GND: track 3.34 -> 54.3 mm, vias 0 -> 58
- net SPI1_SCLK: track 0.00 -> 50.7 mm, vias 0 -> 1
- net SPI0_SCLK: track 0.00 -> 45.4 mm, vias 0 -> 2
- net CC_RSTN: track 0.00 -> 43.5 mm, vias 0 -> 2
- net SPI0_DEV1: track 0.00 -> 43.4 mm, vias 0 -> 2
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- added copper zone on In2.Cu, net 3v3
- added copper zone on B.Cu, net GND
- added copper zone on F.Cu, net GND
- added copper zone on In1.Cu, net GND
Other:
- board text added: "3v3"
- board text added: "Designed by Keyaan Khatri in 2025"
- board text added: "GND"
- board text added: "GP3"
- board text added: "I completed the pcb in 4 hours"
- board text added: "Made By Humans On Earth"
- board text added: "RSTN"
- board text added: "SPI0 MISO"
- board text added: "SPI0 MOSI"
- board text added: "SPI0 SCLK"
